File: avr-attiny412-boosted.sch (KiCad schematic (older format))
At the start: 0 parts

Commit message: Partial schematic
Parts:
- added C?: 10uF, symbol Device:C
- added F?: Polyfuse, symbol Device:Polyfuse
- added J?: BAT_JST_PH, symbol Connector_Generic:Conn_01x02
- added L?: 4.7uH, symbol Device:L
- added R1, R2: 100k, symbol Device:R_Small
- added U1: MCP1640, symbol local_symbols:MCP1640
- added U2: MIC809, symbol local_symbols:MIC809
- added U?: attiny412, symbol local_symbols:attiny412
Connections:
- net labels added: GND, VBAT
- wire segments 0 -> 26
Other:
- note added: "DNP"
- note added: "Place either:\n R2 + MIC809: voltage supervisor enabled\n (useful when using Li-Ion batteries)\nor\n R1: bypass superviser, boost always on\n (useful when using non-rechargeable)"
- note added: "Vth = 2.93V"
Changed lines of the file:
@@
 EESchema Schematic File Version 4
-EELAYER 26 0
+LIBS:avr-attiny412-boosted-cache
+EELAYER 29 0
 EELAYER END
-$Descr A4 11693 8268
+$Descr USLetter 11000 8500
 encoding utf-8
 Sheet 1 1
 Title "AVR ATtiny412 with integrated boost regulator"
-Date "2018-12-02"
+Date "2019-04-03"
 Rev "1"
 Comp ""
@@
 Comment4 ""
 $EndDescr
+$Comp
+L local_symbols:attiny412 U?
+U 1 1 5CA5A3F1
+P 5900 2350
+F 0 "U?" H 5900 3023 50  0000 C CNN
+F 1 "attiny412" H 5900 2930 50  0000 C CNN
+F 2 "" H 6000 2350 50  0001 C CNN
+F 3 "" H 6000 2350 50  0001 C CNN
+	1    5900 2350
+	1    0    0    -1
+$EndComp
+$Comp
+L local_symbols:MCP1640 U1
+U 1 1 5CA5DBC4
+P 4100 2000
+F 0 "U1" H 4150 2500 50  0000 C CNN
+F 1 "MCP1640" H 4250 2400 50  0000 C CNN
+F 2 "" H 4100 2000 50  0001 C CNN
+F 3 "" H 4100 2000 50  0001 C CNN
+	1    4100 2000
+	1    0    0    -1
+$EndComp
+$Comp
+L local_symbols:MIC809 U2
+U 1 1 5CA5EF61
+P 2300 3300
+F 0 "U2" H 2067 3447 50  0000 R CNN
+F 1 "MIC809" H 2067 3354 50  0000 R CNN
+F 2 "" H 2300 3300 50  0001 C CNN
+F 3 "" H 2300 3300 50  0001 C CNN
+	1    2300 3300
+	1    0    0    -1
+$EndComp
+$Comp
+L Device:R_Small R1
+U 1 1 5CA6454D
+P 3350 2050
+F 0 "R1" H 3409 2097 50  0000 L CNN
+F 1 "100k" H 3409 2004 50  0000 L CNN
+F 2 "" H 3350 2050 50  0001 C CNN
+F 3 "~" H 3350 2050 50  0001 C CNN
+	1    3350 2050
+	1    0    0    -1
+$EndComp
+$Comp
+L Device:R_Small R2
+U 1 1 5CA65A2C
+P 3350 2350
+F 0 "R2" H 3409 2397 50  0000 L CNN
+F 1 "100k" H 3409 2304 50  0000 L CNN
+F 2 "" H 3350 2350 50  0001 C CNN
+F 3 "~" H 3350 2350 50  0001 C CNN
+	1    3350 2350
+	1    0    0    -1
+$EndComp
+$Comp
+L power:GND #PWR?
+U 1 1 5CA660DB
+P 3350 2500
+F 0 "#PWR?" H 3350 2250 50  0001 C CNN
+F 1 "GND" H 3354 2321 50  0000 C CNN
+F 2 "" H 3350 2500 50  0001 C CNN
+F 3 "" H 3350 2500 50  0001 C CNN
+	1    3350 2500
+	1    0    0    -1
+$EndComp
+Wire Wire Line
+	3350 2450 3350 2500
+Wire Wire Line
+	3600 2200 3350 2200
+Wire Wire Line
+	3350 2150 3350 2200
+Connection ~ 3350 2200
+Wire Wire Line
+	3350 2200 3350 2250
+Wire Wire Line
+	3350 1900 3350 1950
+$Comp
+L power:GND #PWR?
+U 1 1 5CA67BCF
+P 2300 3600
+F 0 "#PWR?" H 2300 3350 50  0001 C CNN
+F 1 "GND" H 2304 3421 50  0000 C CNN
+F 2 "" H 2300 3600 50  0001 C CNN
+F 3 "" H 2300 3600 50  0001 C CNN
+	1    2300 3600
+	1    0    0    -1
+$EndComp
+Text Notes 3100 3400 0    50   ~ 0
+Place either:\n  R2 + MIC809: voltage supervisor enabled\n  (useful when using Li-Ion batteries)\nor\n  R1: bypass superviser, boost always on\n  (useful when using non-rechargeable)
+$Comp
+L power:GND #PWR?
+U 1 1 5CA680CD
+P 4200 2600
+F 0 "#PWR?" H 4200 2350 50  0001 C CNN
+F 1 "GND" H 4204 2421 50  0000 C CNN
+F 2 "" H 4200 2600 50  0001 C CNN
+F 3 "" H 4200 2600 50  0001 C CNN
+	1    4200 2600
+	1    0    0    -1
+$EndComp
+$Comp
+L Connector_Generic:Conn_01x02 J?
+U 1 1 5CA68B1C
+P 1600 1900
+F 0 "J?" H 1750 1900 50  0000 C CNN
+F 1 "BAT_JST_PH" H 1900 1800 50  0000 C CNN
+F 2 "" H 1600 1900 50  0001 C CNN
+F 3 "~" H 1600 1900 50  0001 C CNN
+	1    1600 1900
+	-1   0    0    -1
+$EndComp
+$Comp
+L Device:Polyfuse F?
+U 1 1 5CA6AFCA
+P 2150 1900
+F 0 "F?" V 1917 1900 50  0000 C CNN
+F 1 "Polyfuse" V 2010 1900 50  0000 C CNN
+F 2 "" H 2200 1700 50  0001 L CNN
+F 3 "~" H 2150 1900 50  0001 C CNN
+	1    2150 1900
+	0    1    1    0
+$EndComp
+Wire Wire Line
+	1800 1900 2000 1900
+Wire Wire Line
+	1800 2000 1900 2000
+Wire Wire Line
+	1900 2000 1900 2100
+$Comp
+L power:GND #PWR?
+U 1 1 5CA6DD23
+P 1900 2100
+F 0 "#PWR?" H 1900 1850 50  0001 C CNN
+F 1 "GND" H 1904 1921 50  0000 C CNN
+F 2 "" H 1900 2100 50  0001 C CNN
+F 3 "" H 1900 2100 50  0001 C CNN
+	1    1900 2100
+	1    0    0    -1
+$EndComp
+Connection ~ 3350 1900
+Wire Wire Line
+	3350 1900 3600 1900
+$Comp
+L Device:C C?
+U 1 1 5CA84421
+P 2600 2200
+F 0 "C?" H 2400 2250 50  0000 L CNN
+F 1 "10uF" H 2300 2150 50  0000 L CNN
+F 2 "" H 2638 2050 50  0001 C CNN
+F 3 "~" H 2600 2200 50  0001 C CNN
+	1    2600 2200
+	1    0    0    -1
+$EndComp
+Connection ~ 2600 1900
+Wire Wire Line
+	2600 1900 3100 1900
+Wire Wire Line
+	2600 1900 2600 2050
+$Comp
+L power:GND #PWR?
+U 1 1 5CA86A14
+P 2600 2500
+F 0 "#PWR?" H 2600 2250 50  0001 C CNN
+F 1 "GND" H 2604 2321 50  0000 C CNN
+F 2 "" H 2600 2500 50  0001 C CNN
+F 3 "" H 2600 2500 50  0001 C CNN
+	1    2600 2500
+	1    0    0    -1
+$EndComp
+Wire Wire Line
+	2600 2350 2600 2500
+Text Notes 3150 2100 0    50   ~ 0
+DNP
+Wire Wire Line
+	4000 1500 4000 1400
+$Comp
+L Device:L L?
+U 1 1 5CA87E91
+P 3550 1400
+F 0 "L?" V 3748 1400 50  0000 C CNN
+F 1 "4.7uH" V 3655 1400 50  0000 C CNN
+F 2 "" H 3550 1400 50  0001 C CNN
+F 3 "~" H 3550 1400 50  0001 C CNN
+	1    3550 1400
+	0    -1   -1   0
+$EndComp
+Wire Wire Line
+	3700 1400 4000 1400
+Wire Wire Line
+	3400 1400 3100 1400
+Wire Wire Line
+	3100 1400 3100 1900
+Connection ~ 3100 1900
+Wire Wire Line
+	3100 1900 3350 1900
+Connection ~ 2500 1900
+Wire Wire Line
+	2500 1900 2600 1900
+Wire Wire Line
+	2300 1900 2500 1900
+Text GLabel 2600 1750 2    50   Input ~ 0
+VBAT
+Wire Wire Line
+	2500 1750 2600 1750
+Wire Wire Line
+	2500 1900 2500 1750
+Text GLabel 2100 2700 0    50   Input ~ 0
+VBAT
+Wire Wire Line
+	2100 2700 2200 2700
+Wire Wire Line
+	2200 2700 2200 2800
+Wire Wire Line
+	2700 3100 3000 3100
+Wire Wire Line
+	3000 3100 3000 2200
+Wire Wire Line
+	3000 2200 3350 2200
+Text Notes 2250 2950 0    50   ~ 0
+Vth = 2.93V
 $EndSCHEMATC

Commit message: Add load switch symbol, and complete schematic (pending validation)
Parts:
- added C2: 4.7uF, symbol Device:C
- added C3, C5: 10uF, symbol Device:C
- added C4: 0.1uF, symbol Device:C_Small
- added J10, J11, J12, J13, J14, J15, J2, J3, J4, J5, J6, J7, J8, J9: Conn_01x01, symbol Connector_Generic:Conn_01x01
- added R3, R4: R, symbol Device:R
- added R5: 3.3k, symbol Device:R
- added R6: 100k, symbol Device:R_Small
- added R7: 1k, symbol Device:R_Small
- added R8, R9: 10k, symbol Device:R_Small
- added SW1: SW_Push, symbol Switch:SW_Push
- added U4: MIC9409x, symbol local_symbols:MIC9409x
- gave numbers to parts that had none: 5
Connections:
- net labels added: PA1, PA2, PA3, PA6, PA7, UPDI, VPP, VSW
- wire segments 26 -> 85
Other:
- note added: "3 pins for\nprogramming"
- note added: "750mA"
- note added: "LED strip with\ndata on PA7"
- note added: "Load switch, controlled\nwith PA6"
- note added: "MCP1640:\n FB = 1.21V\n\nMCP16251\n FB = 1.23V\n\nTPS61070 / TPS61073\n FB = 0.5V"
- note added: "SW1: rest in software\nor other functionality"
- note added: "optional\nI2C pull-ups"

Commit message: Fix LED load capacitor
Connections:
- wire segments 85 -> 86
Other:
- moved on the sheet: C5
Changed lines of the file:
@@
 	1    0    0    -1
 $EndComp
-Text GLabel 9400 4000 0    50   Input ~ 0
+Text GLabel 9100 3900 0    50   Input ~ 0
 VSW
 Text GLabel 9200 4600 0    50   Input ~ 0
@@
 L Device:C C5
 U 1 1 5CB8DCFC
-P 9500 4250
-F 0 "C5" H 9600 4250 50  0000 L CNN
-F 1 "10uF" H 9550 4150 50  0000 L CNN
-F 2 "" H 9538 4100 50  0001 C CNN
-F 3 "~" H 9500 4250 50  0001 C CNN
-	1    9500 4250
+P 9200 4150
+F 0 "C5" H 9300 4150 50  0000 L CNN
+F 1 "10uF" H 9250 4050 50  0000 L CNN
+F 2 "" H 9238 4000 50  0001 C CNN
+F 3 "~" H 9200 4150 50  0001 C CNN
+	1    9200 4150
 	1    0    0    -1
 $EndComp
@@
 	9300 4600 9200 4600
 Wire Wire Line
-	9400 4000 9500 4000
+	9100 3900 9200 3900
 Wire Wire Line
-	9500 4000 9500 4100
-Wire Wire Line
-	9500 4400 9500 4500
+	9200 3900 9200 4000
 Wire Wire Line
 	9500 4500 9600 4500
+$Comp
+L power:GND #PWR?
+U 1 1 5CBBC9A3
+P 9200 4300
+F 0 "#PWR?" H 9200 4050 50  0001 C CNN
+F 1 "GND" H 9200 4150 50  0000 C CNN
+F 2 "" H 9200 4300 50  0001 C CNN
+F 3 "" H 9200 4300 50  0001 C CNN
+	1    9200 4300
+	1    0    0    -1
+$EndComp
+Wire Wire Line
+	9200 3900 9500 3900
+Wire Wire Line
+	9500 3900 9500 4500
+Connection ~ 9200 3900
 $EndSCHEMATC

Commit message: Improve footprints (inductor, JST PH, SC-70-6), add JST BAT schematic symbol
Parts:
- removed J1: BAT_JST_PH, symbol Connector_Generic:Conn_01x02
- added JST_PH_BAT1: JST_PH_BAT, symbol local_symbols:JST_PH_BAT
Changed lines of the file:
@@
-$EndComp
-$Comp
-L Connector_Generic:Conn_01x02 J1
-U 1 1 5CA68B1C
-P 1600 1900
-F 0 "J1" H 1750 1900 50  0000 C CNN
-F 1 "BAT_JST_PH" H 1900 1800 50  0000 C CNN
-F 2 "" H 1600 1900 50  0001 C CNN
-F 3 "~" H 1600 1900 50  0001 C CNN
-	1    1600 1900
-	-1   0    0    -1
 $EndComp
 $Comp
@@
 	9500 3900 9500 4500
 Connection ~ 9200 3900
+$Comp
+L local_symbols:JST_PH_BAT JST_PH_BAT1
+U 1 1 5CBEFBE8
+P 1600 1900
+F 0 "JST_PH_BAT1" H 1550 2050 50  0000 C CNN
+F 1 "JST_PH_BAT" H 1550 1700 50  0001 C CNN
+F 2 "" H 1600 1900 50  0001 C CNN
+F 3 "~" H 1600 1900 50  0001 C CNN
+	1    1600 1900
+	1    0    0    -1
+$EndComp
 $EndSCHEMATC

Commit message: Footprints, minor fixes, footprint assignment, netlist
Parts:
- C1, C2, F1: footprint (none) -> local_footprints:1206_HS
- C3, C5: footprint (none) -> local_footprints:1210_HS
- C4, R1, R2, R3, R4, R5, R6, R7, R8, R9: footprint (none) -> local_footprints:0805_HS
- J10, J11, J12: footprint (none) -> local_footprints:Conn_1-wire
- J13, J14, J15, J2, J3, J4, J5, J6, J7, J8, J9: footprint (none) -> local_footprints:Pin_Header_Straight_1x01_Pitch2.54mm
- JST_PH_BAT1: footprint (none) -> local_footprints:JST_PH_S2B-PH-K_02x2.00mm_Angled_WiderHole
- L1: footprint (none) -> local_footprints:L_Taiyo-Yuden_NR-S-40xx_HS
- SW1: footprint (none) -> local_footprints:SW_SPST_PUSH_6mm_3mm
- U1: footprint (none) -> local_footprints:SOT-23-6_HS
- U2: footprint (none) -> local_footprints:SOT-23_HS
- U3: footprint (none) -> local_footprints:SOIC-8_3.9x4.9mm_Pitch1.27mm_HS
- U4: footprint (none) -> local_footprints:SOT-363_SC-70-6_HS
Other:
- note added: "3 smaller PTHs for\nprogramming"
- note added: "Load switch,\ncontrolled with PA6"
- note added: "Pin-compatible with:\n\n MCP1640:\n FB = 1.21V\n\n MCP16251:\n FB = 1.23V\n\n TPS61070 / TPS61073:\n FB = 0.5V"
- note added: "SW1: reset in software\nor other functionality"
- note added: "push-pull"
- note removed: "3 pins for\nprogramming"
- note removed: "Load switch, controlled\nwith PA6"
- note removed: "MCP1640:\n FB = 1.21V\n\nMCP16251\n FB = 1.23V\n\nTPS61070 / TPS61073\n FB = 0.5V"
- note removed: "SW1: rest in software\nor other functionality"
Changed lines of the file:
@@
 F 0 "U3" H 7600 2873 50  0000 C CNN
 F 1 "attiny412" H 7600 2780 50  0000 C CNN
-F 2 "" H 7700 2200 50  0001 C CNN
+F 2 "local_footprints:SOIC-8_3.9x4.9mm_Pitch1.27mm_HS" H 7700 2200 50  0001 C CNN
 F 3 "" H 7700 2200 50  0001 C CNN
 	1    7600 2200
@@
 F 0 "U1" H 4150 2500 50  0000 C CNN
 F 1 "MCP1640" H 4250 2400 50  0000 C CNN
-F 2 "" H 4100 2000 50  0001 C CNN
+F 2 "local_footprints:SOT-23-6_HS" H 4100 2000 50  0001 C CNN
 F 3 "" H 4100 2000 50  0001 C CNN
 	1    4100 2000
@@
 F 0 "U2" H 2067 3447 50  0000 R CNN
 F 1 "MIC809" H 2067 3354 50  0000 R CNN
-F 2 "" H 2300 3300 50  0001 C CNN
+F 2 "local_footprints:SOT-23_HS" H 2300 3300 50  0001 C CNN
 F 3 "" H 2300 3300 50  0001 C CNN
 	1    2300 3300
@@
 F 0 "R1" H 3409 2097 50  0000 L CNN
 F 1 "100k" H 3409 2004 50  0000 L CNN
-F 2 "" H 3350 2050 50  0001 C CNN
+F 2 "local_footprints:0805_HS" H 3350 2050 50  0001 C CNN
 F 3 "~" H 3350 2050 50  0001 C CNN
 	1    3350 2050
@@
 F 0 "R2" H 3409 2397 50  0000 L CNN
 F 1 "100k" H 3409 2304 50  0000 L CNN
-F 2 "" H 3350 2350 50  0001 C CNN
+F 2 "local_footprints:0805_HS" H 3350 2350 50  0001 C CNN
 F 3 "~" H 3350 2350 50  0001 C CNN
 	1    3350 2350
@@
 F 0 "F1" V 1917 1900 50  0000 C CNN
 F 1 "Polyfuse" V 2010 1900 50  0000 C CNN
-F 2 "" H 2200 1700 50  0001 L CNN
+F 2 "local_footprints:1206_HS" H 2200 1700 50  0001 L CNN
 F 3 "~" H 2150 1900 50  0001 C CNN
 	1    2150 1900
@@
 F 0 "C1" H 2400 2250 50  0000 L CNN
 F 1 "10uF" H 2300 2150 50  0000 L CNN
-F 2 "" H 2638 2050 50  0001 C CNN
+F 2 "local_footprints:1206_HS" H 2638 2050 50  0001 C CNN
 F 3 "~" H 2600 2200 50  0001 C CNN
 	1    2600 2200
@@
 F 0 "L1" V 3748 1400 50  0000 C CNN
 F 1 "4.7uH" V 3655 1400 50  0000 C CNN
-F 2 "" H 3550 1400 50  0001 C CNN
+F 2 "local_footprints:L_Taiyo-Yuden_NR-S-40xx_HS" H 3550 1400 50  0001 C CNN
 F 3 "~" H 3550 1400 50  0001 C CNN
 	1    3550 1400
@@
 F 0 "R3" H 4870 1997 50  0000 L CNN
 F 1 "R" H 4870 1904 50  0000 L CNN
-F 2 "" V 4730 1950 50  0001 C CNN
+F 2 "local_footprints:0805_HS" V 4730 1950 50  0001 C CNN
 F 3 "~" H 4800 1950 50  0001 C CNN
 	1    4800 1950
@@
 F 0 "R4" H 4870 2297 50  0000 L CNN
 F 1 "R" H 4870 2204 50  0000 L CNN
-F 2 "" V 4730 2250 50  0001 C CNN
+F 2 "local_footprints:0805_HS" V 4730 2250 50  0001 C CNN
 F 3 "~" H 4800 2250 50  0001 C CNN
 	1    4800 2250
@@
 F 0 "C2" H 5300 2100 50  0000 L CNN
 F 1 "4.7uF" H 5250 2000 50  0000 L CNN
-F 2 "" H 5238 1950 50  0001 C CNN
+F 2 "local_footprints:1206_HS" H 5238 1950 50  0001 C CNN
 F 3 "~" H 5200 2100 50  0001 C CNN
 	1    5200 2100
@@
 F 0 "C3" H 5700 2100 50  0000 L CNN
 F 1 "10uF" H 5650 2000 50  0000 L CNN
-F 2 "" H 5638 1950 50  0001 C CNN
+F 2 "local_footprints:1210_HS" H 5638 1950 50  0001 C CNN
 F 3 "~" H 5600 2100 50  0001 C CNN
 	1    5600 2100
@@
 Wire Wire Line
 	5200 1800 5600 1800
-Text Notes 4550 1600 0    50   ~ 0
-MCP1640:\n  FB = 1.21V\n\nMCP16251\n  FB = 1.23V\n\nTPS61070 / TPS61073\n  FB = 0.5V
+Text Notes 4400 1550 0    50   ~ 0
+Pin-compatible with:\n\n  MCP1640:\n    FB = 1.21V\n\n  MCP16251:\n    FB = 1.23V\n\n  TPS61070 / TPS61073:\n    FB = 0.5V
 Wire Wire Line
 	5600 1800 5900 1800
@@
 F 0 "C4" H 6750 2100 50  0000 L CNN
 F 1 "0.1uF" H 6700 2000 50  0000 L CNN
-F 2 "" H 7000 2050 50  0001 C CNN
+F 2 "local_footprints:0805_HS" H 7000 2050 50  0001 C CNN
 F 3 "~" H 7000 2050 50  0001 C CNN
 	1    7000 2050
@@
 F 0 "R5" V 8440 2200 50  0000 C CNN
 F 1 "3.3k" V 8533 2200 50  0000 C CNN
-F 2 "" V 8580 2200 50  0001 C CNN
+F 2 "local_footprints:0805_HS" V 8580 2200 50  0001 C CNN
 F 3 "~" H 8650 2200 50  0001 C CNN
 	1    8650 2200
@@
 F 0 "SW1" V 8353 2653 50  0000 L CNN
 F 1 "SW_Push" V 8446 2653 50  0000 L CNN
-F 2 "" H 8400 2700 50  0001 C CNN
+F 2 "local_footprints:SW_SPST_PUSH_6mm_3mm" H 8400 2700 50  0001 C CNN
 F 3 "~" H 8400 2700 50  0001 C CNN
 	1    8400 2500
@@
 	8400 2700 8400 2800
 Text Notes 8550 2850 0    50   ~ 0
-SW1: rest in software\nor other functionality
+SW1: reset in software\nor other functionality
 Text GLabel 4000 4500 2    50   Input ~ 0
 PA1
@@
 F 0 "J3" H 3450 4600 50  0000 C CNN
 F 1 "Conn_01x01" H 3700 4600 50  0001 C CNN
-F 2 "" H 3300 4600 50  0001 C CNN
+F 2 "local_footprints:Pin_Header_Straight_1x01_Pitch2.54mm" H 3300 4600 50  0001 C CNN
 F 3 "~" H 3300 4600 50  0001 C CNN
 	1    3300 4600
@@
 F 0 "J4" H 3450 4700 50  0000 C CNN
 F 1 "Conn_01x01" H 3700 4700 50  0001 C CNN
-F 2 "" H 3300 4700 50  0001 C CNN
+F 2 "local_footprints:Pin_Header_Straight_1x01_Pitch2.54mm" H 3300 4700 50  0001 C CNN
 F 3 "~" H 3300 4700 50  0001 C CNN
 	1    3300 4700
@@
 F 0 "J5" H 3450 4800 50  0000 C CNN
 F 1 "Conn_01x01" H 3700 4800 50  0001 C CNN
-F 2 "" H 3300 4800 50  0001 C CNN
+F 2 "local_footprints:Pin_Header_Straight_1x01_Pitch2.54mm" H 3300 4800 50  0001 C CNN
 F 3 "~" H 3300 4800 50  0001 C CNN
 	1    3300 4800
@@
 F 0 "J2" H 3450 4500 50  0000 C CNN
 F 1 "Conn_01x01" H 3700 4500 50  0001 C CNN
-F 2 "" H 3300 4500 50  0001 C CNN
+F 2 "local_footprints:Pin_Header_Straight_1x01_Pitch2.54mm" H 3300 4500 50  0001 C CNN
 F 3 "~" H 3300 4500 50  0001 C CNN
 	1    3300 4500
@@
 F 0 "R8" H 3500 4300 50  0000 L CNN
 F 1 "10k" H 3500 4200 40  0000 L CNN
-F 2 "" H 3650 4250 50  0001 C CNN
+F 2 "local_footprints:0805_HS" H 3650 4250 50  0001 C CNN
 F 3 "~" H 3650 4250 50  0001 C CNN
 	1    3650 4250
@@
 F 0 "R9" H 3850 4300 50  0000 L CNN
 F 1 "10k" H 3850 4200 40  0000 L CNN
-F 2 "" H 3800 4250 50  0001 C CNN
+F 2 "local_footprints:0805_HS" H 3800 4250 50  0001 C CNN
 F 3 "~" H 3800 4250 50  0001 C CNN
 	1    3800 4250
@@
 F 0 "J9" H 4950 4800 50  0000 C CNN
 F 1 "Conn_01x01" H 5200 4800 50  0001 C CNN
-F 2 "" H 4800 4800 50  0001 C CNN
+F 2 "local_footprints:Pin_Header_Straight_1x01_Pitch2.54mm" H 4800 4800 50  0001 C CNN
 F 3 "~" H 4800 4800 50  0001 C CNN
 	1    4800 4800
@@
 F 0 "J10" H 6150 4500 50  0000 C CNN
 F 1 "Conn_01x01" H 6400 4500 50  0001 C CNN
-F 2 "" H 6000 4500 50  0001 C CNN
+F 2 "local_footprints:Conn_1-wire" H 6000 4500 50  0001 C CNN
 F 3 "~" H 6000 4500 50  0001 C CNN
 	1    6000 4500
@@
 F 0 "J11" H 6150 4600 50  0000 C CNN
 F 1 "Conn_01x01" H 6400 4600 50  0001 C CNN
-F 2 "" H 6000 4600 50  0001 C CNN
+F 2 "local_footprints:Conn_1-wire" H 6000 4600 50  0001 C CNN
 F 3 "~" H 6000 4600 50  0001 C CNN
 	1    6000 4600
@@
 F 0 "J12" H 6150 4700 50  0000 C CNN
 F 1 "Conn_01x01" H 6400 4700 50  0001 C CNN
-F 2 "" H 6000 4700 50  0001 C CNN
+F 2 "local_footprints:Conn_1-wire" H 6000 4700 50  0001 C CNN
 F 3 "~" H 6000 4700 50  0001 C CNN
 	1    6000 4700
@@
 F 0 "J7" H 4950 4600 50  0000 C CNN
 F 1 "Conn_01x01" H 5200 4600 50  0001 C CNN
-F 2 "" H 4800 4600 50  0001 C CNN
+F 2 "local_footprints:Pin_Header_Straight_1x01_Pitch2.54mm" H 4800 4600 50  0001 C CNN
 F 3 "~" H 4800 4600 50  0001 C CNN
 	1    4800 4600
@@
 F 0 "J8" H 4950 4700 50  0000 C CNN
 F 1 "Conn_01x01" H 5200 4700 50  0001 C CNN
-F 2 "" H 4800 4700 50  0001 C CNN
+F 2 "local_footprints:Pin_Header_Straight_1x01_Pitch2.54mm" H 4800 4700 50  0001 C CNN
 F 3 "~" H 4800 4700 50  0001 C CNN
 	1    4800 4700
@@
 F 0 "J6" H 4950 4500 50  0000 C CNN
 F 1 "Conn_01x01" H 5200 4500 50  0001 C CNN
-F 2 "" H 4800 4500 50  0001 C CNN
+F 2 "local_footprints:Pin_Header_Straight_1x01_Pitch2.54mm" H 4800 4500 50  0001 C CNN
 F 3 "~" H 4800 4500 50  0001 C CNN
 	1    4800 4500
@@
 F 0 "U4" H 7850 5173 50  0000 C CNN
 F 1 "MIC9409x" H 7850 5080 50  0000 C CNN
-F 2 "" H 7700 4700 50  0001 C CNN
+F 2 "local_footprints:SOT-363_SC-70-6_HS" H 7700 4700 50  0001 C CNN
 F 3 "" H 7700 4700 50  0001 C CNN
 	1    7900 4700
@@
 F 0 "R6" H 7359 4947 50  0000 L CNN
 F 1 "100k" H 7359 4854 50  0000 L CNN
-F 2 "" H 7300 4900 50  0001 C CNN
+F 2 "local_footprints:0805_HS" H 7300 4900 50  0001 C CNN
 F 3 "~" H 7300 4900 50  0001 C CNN
 	1    7300 4900
@@
 F 0 "J15" H 9950 4700 50  0000 C CNN
 F 1 "Conn_01x01" H 10200 4700 50  0001 C CNN
-F 2 "" H 9800 4700 50  0001 C CNN
+F 2 "local_footprints:Pin_Header_Straight_1x01_Pitch2.54mm" H 9800 4700 50  0001 C CNN
 F 3 "~" H 9800 4700 50  0001 C CNN
 	1    9800 4700
@@
 F 0 "J14" H 9950 4600 50  0000 C CNN
 F 1 "Conn_01x01" H 10200 4600 50  0001 C CNN
-F 2 "" H 9800 4600 50  0001 C CNN
+F 2 "local_footprints:Pin_Header_Straight_1x01_Pitch2.54mm" H 9800 4600 50  0001 C CNN
 F 3 "~" H 9800 4600 50  0001 C CNN
 	1    9800 4600
@@
 F 0 "J13" H 9950 4500 50  0000 C CNN
 F 1 "Conn_01x01" H 10200 4500 50  0001 C CNN
-F 2 "" H 9800 4500 50  0001 C CNN
+F 2 "local_footprints:Pin_Header_Straight_1x01_Pitch2.54mm" H 9800 4500 50  0001 C CNN
 F 3 "~" H 9800 4500 50  0001 C CNN
 	1    9800 4500
@@
 Wire Wire Line
 	9500 4700 9500 4800
-Text Notes 6050 5250 0    50   ~ 0
-3 pins for\nprogramming
+Text Notes 5950 5250 0    50   ~ 0
+3 smaller PTHs for\nprogramming
 Text Notes 7400 5600 0    50   ~ 0
-Load switch, controlled\nwith PA6
+Load switch,\ncontrolled with PA6
 Text Notes 9200 5300 0    50   ~ 0
 LED strip with\ndata on PA7
@@
 F 0 "C5" H 9300 4150 50  0000 L CNN
 F 1 "10uF" H 9250 4050 50  0000 L CNN
-F 2 "" H 9238 4000 50  0001 C CNN
+F 2 "local_footprints:1210_HS" H 9238 4000 50  0001 C CNN
 F 3 "~" H 9200 4150 50  0001 C CNN
 	1    9200 4150
@@
 F 0 "R7" V 9300 4600 50  0000 C CNN
 F 1 "1k" V 9400 4600 35  0000 C CNN
-F 2 "" H 9400 4600 50  0001 C CNN
+F 2 "local_footprints:0805_HS" H 9400 4600 50  0001 C CNN
 F 3 "~" H 9400 4600 50  0001 C CNN
 	1    9400 4600
@@
 	9500 4500 9600 4500
 $Comp
-L power:GND #PWR?
+L power:GND #PWR0101
 U 1 1 5CBBC9A3
 P 9200 4300
-F 0 "#PWR?" H 9200 4050 50  0001 C CNN
+F 0 "#PWR0101" H 9200 4050 50  0001 C CNN
 F 1 "GND" H 9200 4150 50  0000 C CNN
 F 2 "" H 9200 4300 50  0001 C CNN
@@
 F 0 "JST_PH_BAT1" H 1550 2050 50  0000 C CNN
 F 1 "JST_PH_BAT" H 1550 1700 50  0001 C CNN
-F 2 "" H 1600 1900 50  0001 C CNN
+F 2 "local_footprints:JST_PH_S2B-PH-K_02x2.00mm_Angled_WiderHole" H 1600 1900 50  0001 C CNN
 F 3 "~" H 1600 1900 50  0001 C CNN
 	1    1600 1900
 	1    0    0    -1
 $EndComp
+Text Notes 2550 3200 0    50   ~ 0
+push-pull
 $EndSCHEMATC
